File: LED_Bar_Clock.sch (KiCad schematic (older format))
At the start: 50 parts

Commit message: Finalize USB and Power, and update LED layout
- add usb circuitry
  - esd protection w/ varistors
  - logic level shifting w/ zener diodes
  - usb protocol pullup/down resistors
  - usb series data resistors
- update LED layout (now 6-3-5)
- power PTC fuse
Parts:
- removed C? (x4): 104, symbol Device:C_Small
- removed D? (x4): SK6812, LED_SMD:LED_SK6812_PLCC4_5.0x5.0mm_P3.2mm, symbol LED:SK6812
- added D? (x2): 3.6v, symbol Device:D_Zener
- added F?: 500mA PTC, symbol Device:Polyfuse_Small
- added R?: 1.5k, symbol Device:R
- added R?: 5.1k, symbol Device:R
- added R? (x2): 68, symbol Device:R_Small
- added RV? (x2): 5V, symbol Device:Varistor
- C?: value CP -> 226
- J?: value USB_C_Receptacle_USB2.0 -> USB2.0 Type C Receptacle
Connections:
- wire segments 190 -> 191
Other:
- moved on the sheet: BT?, C?, D?, J?, R?, SW?, U?, Y?

Commit message: modify resistor values
changed i2c and reset pullups to 5.1k to match usb cc pulldown.
allows for easier sourcing of parts
Parts:
- R? (x2): value 4.7k -> 5.1k
- R?: value 10k -> 5.1k
Changed lines of the file:
@@
 P 3150 6050
 F 0 "R?" V 2943 6050 50  0000 C CNN
-F 1 "4.7k" V 3034 6050 50  0000 C CNN
+F 1 "5.1k" V 3034 6050 50  0000 C CNN
 F 2 "" V 3080 6050 50  0001 C CNN
 F 3 "~" H 3150 6050 50  0001 C CNN
@@
 P 3150 5550
 F 0 "R?" V 2943 5550 50  0000 C CNN
-F 1 "4.7k" V 3034 5550 50  0000 C CNN
+F 1 "5.1k" V 3034 5550 50  0000 C CNN
 F 2 "" V 3080 5550 50  0001 C CNN
 F 3 "~" H 3150 5550 50  0001 C CNN
@@
 P 3700 4400
 F 0 "R?" H 3759 4446 50  0000 L CNN
-F 1 "10k" H 3759 4355 50  0000 L CNN
+F 1 "5.1k" H 3759 4355 50  0000 L CNN
 F 2 "" H 3700 4400 50  0001 C CNN
 F 3 "~" H 3700 4400 50  0001 C CNN
