File: LED_Bar_Clock_2_Side_SMD.kicad_pcb (KiCad board)
At the start: 2 copper layers, 100 x 100 mm, 52 parts, among them J1 U262-16XN-4BVC11, J2 AVR-ISP-6, SW1 SKHMQKE010, SW2 SW_5_Way, U1 ATtiny84A-SSUR, U2 DS1307Z+, Y1 32.768 kHz

Commit message: fix annotations and silkscreen locations
Parts:
- renumbered C11 to C10, C12 to C11, C13 to C12, C14 to C13, C15 to C14, C16 to C15, C17 to C16, C3 to C2, C4 to C3, C5 to C4, C6 to C5, C7 to C6, C8 to C7, C9 to C8, C10 to C9
Changed lines of the file:
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@@
-(kicad_pcb (version 20171130) (host pcbnew "(5.1.2)-1")
+(kicad_pcb (version 20171130) (host pcbnew 5.1.2)
   (general
     (thickness 1.6)
@@
     (46 B.CrtYd user)
     (47 F.CrtYd user)
-    (48 B.Fab user)
+    (48 B.Fab user hide)
     (49 F.Fab user)
   )
@@
     (zone_connect 2)
     (attr virtual)
-    (fp_text reference REF** (at 0 -4.2) (layer F.SilkS)
+    (fp_text reference REF** (at 0 -4.2) (layer F.SilkS) hide
       (effects (font (size 1 1) (thickness 0.15)))
     )
@@
     (zone_connect 2)
     (attr virtual)
-    (fp_text reference REF** (at 0 -4.2) (layer F.SilkS)
+    (fp_text reference REF** (at 0 -4.2) (layer F.SilkS) hide
       (effects (font (size 1 1) (thickness 0.15)))
     )
@@
   (module Clock_Footprints:K1-5203UA-01 (layer B.Cu)
     (at 100.6 70 315)
-    (fp_text reference SW2 (at 0.059999 0 315) (layer B.SilkS)
+    (fp_text reference SW2 (at 0.059999 0) (layer B.SilkS)
       (effects (font (size 1 1) (thickness 0.15)) (justify mirror))
     )
@@
     (descr "CR2032 Battery Holder, https://datasheet.lcsc.com/szlcsc/Q-J-BS-2-1_C70376.pdf")
     (tags "CR2032 battery holder clip")
-    (fp_text reference BT1 (at 0 -1.27) (layer B.SilkS)
+    (fp_text reference BT1 (at 0 0) (layer B.SilkS)
       (effects (font (size 1 1) (thickness 0.15)) (justify mirror))
     )
@@
     (tags "capacitor handsolder")
     (attr smd)
-    (fp_text reference C3 (at 0 1.43) (layer B.SilkS)
+    (fp_text reference C2 (at -0.125 -1.5) (layer B.SilkS)
       (effects (font (size 1 1) (thickness 0.15)) (justify mirror))
     )
@@
     (tags "capacitor handsolder")
     (attr smd)
-    (fp_text reference C4 (at 0 1.43 180) (layer B.SilkS)
+    (fp_text reference C3 (at 0 1.43 180) (layer B.SilkS)
       (effects (font (size 1 1) (thickness 0.15)) (justify mirror))
     )
@@
     (tags "capacitor handsolder")
     (attr smd)
-    (fp_text reference C5 (at 0 1.43 180) (layer B.SilkS)
+    (fp_text reference C4 (at 0 1.43 180) (layer B.SilkS)
       (effects (font (size 1 1) (thickness 0.15)) (justify mirror))
     )
@@
     (tags "capacitor handsolder")
     (attr smd)
-    (fp_text reference C6 (at 0 1.43 180) (layer B.SilkS)
+    (fp_text reference C5 (at 0 1.43 180) (layer B.SilkS)
       (effects (font (size 1 1) (thickness 0.15)) (justify mirror))
     )
@@
     (tags "capacitor handsolder")
     (attr smd)
-    (fp_text reference C7 (at 0 1.43 180) (layer B.SilkS)
+    (fp_text reference C6 (at 0 1.43 180) (layer B.SilkS)
       (effects (font (size 1 1) (thickness 0.15)) (justify mirror))
     )
@@
     (tags "capacitor handsolder")
     (attr smd)
-    (fp_text reference C8 (at 0 1.43 180) (layer B.SilkS)
+    (fp_text reference C7 (at 0 1.43 180) (layer B.SilkS)
       (effects (font (size 1 1) (thickness 0.15)) (justify mirror))
     )
@@
     (tags "capacitor handsolder")
     (attr smd)
-    (fp_text reference C9 (at 0 1.43 180) (layer B.SilkS)
+    (fp_text reference C8 (at 0 1.43 180) (layer B.SilkS)
       (effects (font (size 1 1) (thickness 0.15)) (justify mirror))
     )
@@
     (tags "capacitor handsolder")
     (attr smd)
-    (fp_text reference C10 (at 0 1.43) (layer B.SilkS)
+    (fp_text reference C9 (at 0 1.43) (layer B.SilkS)
       (effects (font (size 1 1) (thickness 0.15)) (justify mirror))
     )
@@
     (tags "capacitor handsolder")
     (attr smd)
-    (fp_text reference C11 (at 0 1.43) (layer B.SilkS)
+    (fp_text reference C10 (at 0 1.43) (layer B.SilkS)
       (effects (font (size 1 1) (thickness 0.15)) (justify mirror))
     )
@@
     (tags "capacitor handsolder")
     (attr smd)
-    (fp_text reference C12 (at 0 1.43) (layer B.SilkS)
+    (fp_text reference C11 (at 0 1.43) (layer B.SilkS)
       (effects (font (size 1 1) (thickness 0.15)) (justify mirror))
     )
@@
     (tags "capacitor handsolder")
     (attr smd)
-    (fp_text reference C13 (at 0 1.43) (layer B.SilkS)
+    (fp_text reference C12 (at 0 1.43) (layer B.SilkS)
       (effects (font (size 1 1) (thickness 0.15)) (justify mirror))
     )
@@
     (tags "capacitor handsolder")
     (attr smd)
-    (fp_text reference C14 (at 0 1.43) (layer B.SilkS)
+    (fp_text reference C13 (at 0 1.43) (layer B.SilkS)
       (effects (font (size 1 1) (thickness 0.15)) (justify mirror))
     )
@@
     (tags "capacitor handsolder")
     (attr smd)
-    (fp_text reference C15 (at 0 1.43) (layer B.SilkS)
+    (fp_text reference C14 (at 0 1.43) (layer B.SilkS)
       (effects (font (size 1 1) (thickness 0.15)) (justify mirror))
     )
@@
     (tags "capacitor handsolder")
     (attr smd)
-    (fp_text reference C16 (at 0 1.43) (layer B.SilkS)
+    (fp_text reference C15 (at 0 1.43) (layer B.SilkS)
       (effects (font (size 1 1) (thickness 0.15)) (justify mirror))
     )
@@
     (tags "capacitor handsolder")
     (attr smd)
-    (fp_text reference C17 (at 0 1.43) (layer B.SilkS)
+    (fp_text reference C16 (at 0 1.43) (layer B.SilkS)
       (effects (font (size 1 1) (thickness 0.15)) (justify mirror))
     )
@@
     (tags SOD-123)
     (attr smd)
-    (fp_text reference D1 (at 0 2 270) (layer B.SilkS)
+    (fp_text reference D1 (at 0 -2 270) (layer B.SilkS)
       (effects (font (size 1 1) (thickness 0.15)) (justify mirror))
     )
@@
     (tags "resistor handsolder")
     (attr smd)
-    (fp_text reference R1 (at 0 1.43) (layer B.SilkS)
+    (fp_text reference R1 (at 0 -1.5) (layer B.SilkS)
       (effects (font (size 1 1) (thickness 0.15)) (justify mirror))
     )
@@
     (tags "resistor handsolder")
     (attr smd)
-    (fp_text reference R2 (at 0 1.43) (layer B.SilkS)
+    (fp_text reference R2 (at 0 1.5) (layer B.SilkS)
       (effects (font (size 1 1) (thickness 0.15)) (justify mirror))
     )
@@
     (tags "resistor handsolder")
     (attr smd)
-    (fp_text reference R3 (at 0 1.43) (layer B.SilkS)
+    (fp_text reference R3 (at 0 1.5) (layer B.SilkS)
       (effects (font (size 1 1) (thickness 0.15)) (justify mirror))
     )
@@
     (tags "resistor handsolder")
     (attr smd)
-    (fp_text reference R4 (at 0 1.43) (layer B.SilkS)
+    (fp_text reference R4 (at 0 -1.5) (layer B.SilkS)
       (effects (font (size 1 1) (thickness 0.15)) (justify mirror))
     )
@@
     (tags "resistor handsolder")
     (attr smd)
-    (fp_text reference R5 (at 0 1.43 90) (layer B.SilkS)
+    (fp_text reference R5 (at 0 1.5 180) (layer B.SilkS)
       (effects (font (size 1 1) (thickness 0.15)) (justify mirror))
     )
@@
     (tags "resistor handsolder")
     (attr smd)
-    (fp_text reference RV1 (at 0 1.43 270) (layer B.SilkS)
+    (fp_text reference RV1 (at -0.125 1.5 270) (layer B.SilkS)
       (effects (font (size 1 1) (thickness 0.15)) (justify mirror))
     )
@@
     (tags "resistor handsolder")
     (attr smd)
-    (fp_text reference RV2 (at 0 1.43 270) (layer B.SilkS)
+    (fp_text reference RV2 (at -0.125 -1.5 270) (layer B.SilkS)
       (effects (font (size 1 1) (thickness 0.15)) (justify mirror))
     )
@@
     (descr "Crystal THT DS26 6.0mm length 2.0mm diameter http://www.microcrystal.com/images/_Product-Documentation/03_TF_metal_Packages/01_Datasheet/DS-Series.pdf")
     (tags ['DS26'])
-    (fp_text reference Y1 (at -1.57 -1.625 270) (layer B.SilkS)
-      (effects (font (size 1 1) (thickness 0.15)) (justify mirror))
-    )
+    (fp_text reference Y1 (at 0.9 -5 270) (layer B.SilkS)
+      (effects (font (size 1 1) (thickness 0.15)) (justify mirror))
+    )
